Commit message: arm: redesign geometry — real robot morphology, not a cylinder worm
- visible motor housing at every joint (cylinder aligned to rotation axis),
  boxy link segments, wider ribbed base, 2-finger gripper
- two-tone materials (light links, dark joint housings, orange accents)
- joint names/kinematics unchanged → MoveIt config + pick-place loop work
  as-is; verified rendering in RViz, looping live

Co-Authored-By: Claude Fable 5 <noreply@anthropic.com>

File: ros2/robot_arm_description/urdf/robot_arm.urdf.xacro (robot description, xacro)
@@ -1,116 +1,151 @@
 <?xml version="1.0"?>
-<!-- Starter 6-DOF robot arm. Replace the box/cylinder <geometry> with your
-     3D-printed meshes (STL from FreeCAD) as the design firms up; tune the
-     link lengths / joint limits below. This is a working skeleton, not a
-     final design. -->
+<!-- 6-DOF articulated robot arm — proper morphology: a wide base, a visible
+     motor housing at every joint (the cylinders you see at shoulder/elbow/
+     wrist), boxy link segments between them, and a 2-finger gripper.
+     Joint names (joint1..6) are unchanged so the MoveIt config + pick-place
+     loop keep working. Replace <geometry> with your 3D-printed STL meshes
+     and tune the lengths below as the real design firms up. -->
 <robot name="robot_arm" xmlns:xacro="http://www.ros.org/wiki/xacro">
-  <!-- ============ tunable parameters ============ -->
-  <xacro:property name="base_h"   value="0.06"/>   <!-- base height -->
-  <xacro:property name="l1"       value="0.14"/>   <!-- shoulder link -->
-  <xacro:property name="l2"       value="0.16"/>   <!-- upper arm -->
-  <xacro:property name="l3"       value="0.14"/>   <!-- forearm -->
-  <xacro:property name="l4"       value="0.08"/>   <!-- wrist -->
-  <xacro:property name="r"        value="0.03"/>   <!-- link radius -->
-  <xacro:property name="jlim"     value="2.9"/>    <!-- ±rad joint limit -->
-  <xacro:property name="effort"   value="20.0"/>
-  <xacro:property name="vel"      value="2.0"/>
-  <material name="accent"><color rgba="0.85 0.47 0.34 1.0"/></material>
-  <material name="dark">  <color rgba="0.15 0.15 0.17 1.0"/></material>
-  <!-- reusable cylinder link with inertia (needed by ros2_control/gazebo) -->
-  <xacro:macro name="arm_link" params="name length material:=accent">
-    <link name="${name}">
-      <visual>
-        <origin xyz="0 0 ${length/2}" rpy="0 0 0"/>
-        <geometry><cylinder radius="${r}" length="${length}"/></geometry>
-        <material name="${material}"/>
-      </visual>
-      <collision>
-        <origin xyz="0 0 ${length/2}" rpy="0 0 0"/>
-        <geometry><cylinder radius="${r}" length="${length}"/></geometry>
-      </collision>
-      <inertial>
-        <origin xyz="0 0 ${length/2}"/>
-        <mass value="0.5"/>
-        <inertia ixx="0.001" iyy="0.001" izz="0.001" ixy="0" ixz="0" iyz="0"/>
-      </inertial>
-    </link>
+  <!-- ===== tunable lengths (metres) ===== -->
+  <xacro:property name="waist_h" value="0.08"/>
+  <xacro:property name="upper"   value="0.18"/>   <!-- upper arm -->
+  <xacro:property name="fore"    value="0.15"/>   <!-- forearm -->
+  <xacro:property name="wrist"   value="0.06"/>
+  <xacro:property name="jlim"    value="2.9"/>
+  <xacro:property name="pi2"     value="1.5708"/>
+  <material name="link_mat"><color rgba="0.90 0.90 0.92 1"/></material>
+  <material name="joint_mat"><color rgba="0.17 0.17 0.20 1"/></material>
+  <material name="accent"><color rgba="0.85 0.47 0.34 1"/></material>
+  <!-- a motor housing: a cylinder oriented along the joint's rotation axis
+       (rpy picks the axis: z=default, y="pi2 0 0", x="0 pi2 0") -->
+  <xacro:macro name="motor" params="radius len rpy:='0 0 0' mat:=joint_mat">
+    <visual>
+      <origin xyz="0 0 0" rpy="${rpy}"/>
+      <geometry><cylinder radius="${radius}" length="${len}"/></geometry>
+      <material name="${mat}"/>
+    </visual>
+    <collision>
+      <origin xyz="0 0 0" rpy="${rpy}"/>
+      <geometry><cylinder radius="${radius}" length="${len}"/></geometry>
+    </collision>
   </xacro:macro>
-  <!-- ============ world anchor ============ -->
+  <!-- a link segment: a tapered box running from the joint (+Z) to the next -->
+  <xacro:macro name="segment" params="w len mat:=link_mat">
+    <visual>
+      <origin xyz="0 0 ${len/2}"/>
+      <geometry><box size="${w} ${w} ${len}"/></geometry>
+      <material name="${mat}"/>
+    </visual>
+    <collision>
+      <origin xyz="0 0 ${len/2}"/>
+      <geometry><box size="${w} ${w} ${len}"/></geometry>
+    </collision>
+  </xacro:macro>
+  <xacro:macro name="inertia_box" params="mass">
+    <inertial><mass value="${mass}"/>
+      <inertia ixx="0.002" iyy="0.002" izz="0.002" ixy="0" ixz="0" iyz="0"/>
+    </inertial>
+  </xacro:macro>
+  <!-- ===== base ===== -->
   <link name="world"/>
   <link name="base_link">
     <visual>
-      <origin xyz="0 0 ${base_h/2}"/>
-      <geometry><cylinder radius="0.06" length="${base_h}"/></geometry>
-      <material name="dark"/>
+      <origin xyz="0 0 0.015"/>
+      <geometry><cylinder radius="0.08" length="0.03"/></geometry>
+      <material name="joint_mat"/>
     </visual>
-    <collision>
-      <origin xyz="0 0 ${base_h/2}"/>
-      <geometry><cylinder radius="0.06" length="${base_h}"/></geometry>
-    </collision>
-    <inertial><mass value="1.0"/>
-      <inertia ixx="0.002" iyy="0.002" izz="0.002" ixy="0" ixz="0" iyz="0"/>
-    </inertial>
+    <visual>   <!-- riser -->
+      <origin xyz="0 0 0.05"/>
+      <geometry><cylinder radius="0.055" length="0.05"/></geometry>
+      <material name="link_mat"/>
+    </visual>
+    <collision><origin xyz="0 0 0.03"/>
+      <geometry><cylinder radius="0.08" length="0.06"/></geometry></collision>
+    <xacro:inertia_box mass="1.5"/>
   </link>
   <joint name="world_to_base" type="fixed">
     <parent link="world"/><child link="base_link"/>
   </joint>
-  <!-- ============ the 6 links ============ -->
-  <xacro:arm_link name="link1" length="${l1}"/>
-  <xacro:arm_link name="link2" length="${l2}"/>
-  <xacro:arm_link name="link3" length="${l3}"/>
-  <xacro:arm_link name="link4" length="${l4}"/>
-  <xacro:arm_link name="link5" length="0.05"/>
-  <link name="tool0">   <!-- end-effector mount flange -->
-    <visual>
-      <geometry><box size="0.04 0.04 0.02"/></geometry>
-      <material name="dark"/>
-    </visual>
-    <inertial><mass value="0.1"/>
-      <inertia ixx="0.0001" iyy="0.0001" izz="0.0001" ixy="0" ixz="0" iyz="0"/>
-    </inertial>
+  <!-- ===== joint1 waist (Z) ===== -->
+  <link name="link1">
+    <xacro:motor radius="0.055" len="${waist_h}"/>   <!-- vertical waist can -->
+    <visual><origin xyz="0.03 0 ${waist_h*0.6}" rpy="0 ${pi2} 0"/>
+      <geometry><cylinder radius="0.045" length="0.09"/></geometry>
+      <material name="link_mat"/></visual>   <!-- shoulder yoke -->
+    <xacro:inertia_box mass="0.8"/>
   </link>
-  <!-- ============ the 6 joints (waist,shoulder,elbow,3x wrist) ============ -->
-  <joint name="joint1" type="revolute">   <!-- waist: rotate about Z -->
+  <joint name="joint1" type="revolute">
     <parent link="base_link"/><child link="link1"/>
-    <origin xyz="0 0 ${base_h}"/>
-    <axis xyz="0 0 1"/>
-    <limit lower="-${jlim}" upper="${jlim}" effort="${effort}" velocity="${vel}"/>
+    <origin xyz="0 0 0.075"/><axis xyz="0 0 1"/>
+    <limit lower="-${jlim}" upper="${jlim}" effort="30" velocity="2.0"/>
   </joint>
-  <joint name="joint2" type="revolute">   <!-- shoulder: pitch about Y -->
+  <!-- ===== joint2 shoulder (Y) ===== -->
+  <link name="link2">
+    <xacro:motor radius="0.05" len="0.11" rpy="${pi2} 0 0" mat="accent"/>
+    <xacro:segment w="0.055" len="${upper}"/>
+    <xacro:inertia_box mass="0.8"/>
+  </link>
+  <joint name="joint2" type="revolute">
     <parent link="link1"/><child link="link2"/>
-    <origin xyz="0 0 ${l1}"/>
-    <axis xyz="0 1 0"/>
-    <limit lower="-${jlim}" upper="${jlim}" effort="${effort}" velocity="${vel}"/>
+    <origin xyz="0 0 ${waist_h}"/><axis xyz="0 1 0"/>
+    <limit lower="-${jlim}" upper="${jlim}" effort="30" velocity="2.0"/>
   </joint>
-  <joint name="joint3" type="revolute">   <!-- elbow: pitch about Y -->
+  <!-- ===== joint3 elbow (Y) ===== -->
+  <link name="link3">
+    <xacro:motor radius="0.042" len="0.095" rpy="${pi2} 0 0" mat="accent"/>
+    <xacro:segment w="0.045" len="${fore}"/>
+    <xacro:inertia_box mass="0.6"/>
+  </link>
+  <joint name="joint3" type="revolute">
     <parent link="link2"/><child link="link3"/>
-    <origin xyz="0 0 ${l2}"/>
-    <axis xyz="0 1 0"/>
-    <limit lower="-${jlim}" upper="${jlim}" effort="${effort}" velocity="${vel}"/>
+    <origin xyz="0 0 ${upper}"/><axis xyz="0 1 0"/>
+    <limit lower="-${jlim}" upper="${jlim}" effort="20" velocity="2.0"/>
   </joint>
-  <joint name="joint4" type="revolute">   <!-- wrist roll: about Z -->
+  <!-- ===== joint4 wrist roll (Z) ===== -->
+  <link name="link4">
+    <xacro:motor radius="0.036" len="0.07"/>
+    <xacro:segment w="0.04" len="${wrist}" mat="link_mat"/>
+    <xacro:inertia_box mass="0.3"/>
+  </link>
+  <joint name="joint4" type="revolute">
     <parent link="link3"/><child link="link4"/>
-    <origin xyz="0 0 ${l3}"/>
-    <axis xyz="0 0 1"/>
-    <limit lower="-${jlim}" upper="${jlim}" effort="${effort}" velocity="${vel}"/>
+    <origin xyz="0 0 ${fore}"/><axis xyz="0 0 1"/>
+    <limit lower="-${jlim}" upper="${jlim}" effort="10" velocity="2.5"/>
   </joint>
-  <joint name="joint5" type="revolute">   <!-- wrist pitch: about Y -->
+  <!-- ===== joint5 wrist pitch (Y) ===== -->
+  <link name="link5">
+    <xacro:motor radius="0.034" len="0.07" rpy="${pi2} 0 0" mat="accent"/>
+    <xacro:segment w="0.035" len="0.05" mat="link_mat"/>
+    <xacro:inertia_box mass="0.2"/>
+  </link>
+  <joint name="joint5" type="revolute">
     <parent link="link4"/><child link="link5"/>
-    <origin xyz="0 0 ${l4}"/>
-    <axis xyz="0 1 0"/>
-    <limit lower="-${jlim}" upper="${jlim}" effort="${effort}" velocity="${vel}"/>
+    <origin xyz="0 0 ${wrist}"/><axis xyz="0 1 0"/>
+    <limit lower="-${jlim}" upper="${jlim}" effort="10" velocity="2.5"/>
   </joint>
-  <joint name="joint6" type="revolute">   <!-- wrist roll: about Z -->
+  <!-- ===== joint6 tool roll (Z) + gripper ===== -->
+  <link name="tool0">
+    <xacro:motor radius="0.03" len="0.03"/>       <!-- flange -->
+    <visual><origin xyz="0 0 0.03"/>              <!-- gripper palm -->
+      <geometry><box size="0.07 0.03 0.03"/></geometry>
+      <material name="joint_mat"/></visual>
+    <visual><origin xyz="0.028 0 0.065"/>         <!-- finger + -->
+      <geometry><box size="0.014 0.025 0.05"/></geometry>
+      <material name="link_mat"/></visual>
+    <visual><origin xyz="-0.028 0 0.065"/>        <!-- finger - -->
+      <geometry><box size="0.014 0.025 0.05"/></geometry>
+      <material name="link_mat"/></visual>
+    <collision><origin xyz="0 0 0.04"/>
+      <geometry><box size="0.07 0.04 0.08"/></geometry></collision>
+    <xacro:inertia_box mass="0.2"/>
+  </link>
+  <joint name="joint6" type="revolute">
     <parent link="link5"/><child link="tool0"/>
-    <origin xyz="0 0 0.05"/>
-    <axis xyz="0 0 1"/>
-    <limit lower="-${jlim}" upper="${jlim}" effort="${effort}" velocity="${vel}"/>
+    <origin xyz="0 0 0.05"/><axis xyz="0 0 1"/>
+    <limit lower="-${jlim}" upper="${jlim}" effort="10" velocity="2.5"/>
   </joint>
-  <!-- ============ ros2_control: mock hardware for now ============ -->
-  <!-- swap mock_components/GenericSystem for your real servo driver later -->
+  <!-- ===== ros2_control: mock hardware (swap for real servos later) ===== -->
   <ros2_control name="arm_hw" type="system">
-    <hardware>
-      <plugin>mock_components/GenericSystem</plugin>
-    </hardware>
+    <hardware><plugin>mock_components/GenericSystem</plugin></hardware>
     <xacro:macro name="ji" params="name">
       <joint name="${name}">
@@ -120,10 +155,6 @@
       </joint>
     </xacro:macro>
-    <xacro:ji name="joint1"/>
-    <xacro:ji name="joint2"/>
-    <xacro:ji name="joint3"/>
-    <xacro:ji name="joint4"/>
-    <xacro:ji name="joint5"/>
-    <xacro:ji name="joint6"/>
+    <xacro:ji name="joint1"/><xacro:ji name="joint2"/><xacro:ji name="joint3"/>
+    <xacro:ji name="joint4"/><xacro:ji name="joint5"/><xacro:ji name="joint6"/>
   </ros2_control>
 </robot>
