Commit message: weld_cell: fix arm geometry — was a degraded worm, now matches the good arm
- weld_arm.xacro rebuilt to the SAME proper morphology as the standalone
  robot_arm (ribbed base, shoulder yoke, motor housing per joint, boxy
  segments incl. link5, two-tone) — the cell version had been simplified
  and looked thin/worm-like
- renamed macro param 'len' -> 'ln' (xacro warns/errors: shadows builtin)
- single_arm.urdf.xacro validation view added

Co-Authored-By: Claude Fable 5 <noreply@anthropic.com>

File: ros2/weld_cell/urdf/weld_arm.xacro (robot description, xacro)
@@ -1,12 +1,34 @@
 <?xml version="1.0"?>
-<!-- Reusable 6-DOF welding arm as a macro. Instantiate several times with
-     different prefixes + base placements to build a multi-robot cell.
-     Each arm carries a torch on its flange (tool0). -->
+<!-- Reusable 6-DOF welding arm — same proper morphology as the standalone
+     robot_arm (ribbed base, a motor housing at every joint, boxy link
+     segments, two-tone), plus a torch on the flange. Instantiate several
+     times with different prefixes to build a multi-robot cell. -->
 <robot xmlns:xacro="http://www.ros.org/wiki/xacro">
   <material name="wc_link"><color rgba="0.90 0.90 0.92 1"/></material>
   <material name="wc_joint"><color rgba="0.17 0.17 0.20 1"/></material>
   <material name="wc_accent"><color rgba="0.85 0.47 0.34 1"/></material>
-  <material name="wc_torch"><color rgba="0.12 0.12 0.14 1"/></material>
+  <material name="wc_torch"><color rgba="0.10 0.10 0.12 1"/></material>
   <material name="wc_copper"><color rgba="0.72 0.45 0.20 1"/></material>
+  <!-- a motor housing: cylinder aligned to a joint axis (rpy picks the axis) -->
+  <xacro:macro name="wc_motor" params="radius ln rpy:='0 0 0' mat:=wc_joint">
+    <visual><origin xyz="0 0 0" rpy="${rpy}"/>
+      <geometry><cylinder radius="${radius}" length="${ln}"/></geometry>
+      <material name="${mat}"/></visual>
+    <collision><origin xyz="0 0 0" rpy="${rpy}"/>
+      <geometry><cylinder radius="${radius}" length="${ln}"/></geometry></collision>
+  </xacro:macro>
+  <!-- a link segment: a box running from the joint (+Z) to the next -->
+  <xacro:macro name="wc_seg" params="w ln mat:=wc_link">
+    <visual><origin xyz="0 0 ${ln/2}"/>
+      <geometry><box size="${w} ${w} ${ln}"/></geometry>
+      <material name="${mat}"/></visual>
+    <collision><origin xyz="0 0 ${ln/2}"/>
+      <geometry><box size="${w} ${w} ${ln}"/></geometry></collision>
+  </xacro:macro>
+  <xacro:macro name="wc_inertia" params="mass">
+    <inertial><mass value="${mass}"/>
+      <inertia ixx="0.002" iyy="0.002" izz="0.002" ixy="0" ixz="0" iyz="0"/>
+    </inertial>
+  </xacro:macro>
   <xacro:macro name="weld_arm" params="prefix parent x y z yaw color:=wc_accent">
     <xacro:property name="pi2" value="1.5708"/>
@@ -16,14 +38,9 @@
     <xacro:property name="wrist" value="0.06"/>
     <xacro:property name="jl" value="2.9"/>
-    <xacro:macro name="ibox" params="mass">
-      <inertial><mass value="${mass}"/>
-        <inertia ixx="0.002" iyy="0.002" izz="0.002" ixy="0" ixz="0" iyz="0"/>
-      </inertial>
-    </xacro:macro>
-    <!-- fix the arm base to the world/table at (x,y,z) -->
     <joint name="${prefix}anchor" type="fixed">
       <parent link="${parent}"/><child link="${prefix}base_link"/>
       <origin xyz="${x} ${y} ${z}" rpy="0 0 ${yaw}"/>
     </joint>
+    <!-- ribbed base + riser -->
     <link name="${prefix}base_link">
       <visual><origin xyz="0 0 0.015"/>
@@ -35,11 +52,13 @@
       <collision><origin xyz="0 0 0.03"/>
         <geometry><cylinder radius="0.08" length="0.06"/></geometry></collision>
-      <xacro:ibox mass="1.5"/>
+      <xacro:wc_inertia mass="1.5"/>
     </link>
+    <!-- joint1 waist (Z): waist can + shoulder yoke -->
     <link name="${prefix}link1">
-      <visual><geometry><cylinder radius="0.055" length="${waist_h}"/></geometry>
-        <material name="wc_joint"/></visual>
-      <collision><geometry><cylinder radius="0.055" length="${waist_h}"/></geometry></collision>
-      <xacro:ibox mass="0.8"/>
+      <xacro:wc_motor radius="0.055" ln="${waist_h}"/>
+      <visual><origin xyz="0.03 0 ${waist_h*0.6}" rpy="0 ${pi2} 0"/>
+        <geometry><cylinder radius="0.045" length="0.09"/></geometry>
+        <material name="wc_link"/></visual>
+      <xacro:wc_inertia mass="0.8"/>
     </link>
     <joint name="${prefix}joint1" type="revolute">
@@ -48,14 +67,9 @@
       <limit lower="-${jl}" upper="${jl}" effort="30" velocity="2.0"/>
     </joint>
+    <!-- joint2 shoulder (Y): shoulder motor + upper arm -->
     <link name="${prefix}link2">
-      <visual><origin rpy="${pi2} 0 0"/>
-        <geometry><cylinder radius="0.05" length="0.11"/></geometry>
-        <material name="${color}"/></visual>
-      <visual><origin xyz="0 0 ${upper/2}"/>
-        <geometry><box size="0.055 0.055 ${upper}"/></geometry>
-        <material name="wc_link"/></visual>
-      <collision><origin xyz="0 0 ${upper/2}"/>
-        <geometry><box size="0.055 0.055 ${upper}"/></geometry></collision>
-      <xacro:ibox mass="0.8"/>
+      <xacro:wc_motor radius="0.05" ln="0.11" rpy="${pi2} 0 0" mat="${color}"/>
+      <xacro:wc_seg w="0.055" ln="${upper}"/>
+      <xacro:wc_inertia mass="0.8"/>
     </link>
     <joint name="${prefix}joint2" type="revolute">
@@ -64,14 +78,9 @@
       <limit lower="-${jl}" upper="${jl}" effort="30" velocity="2.0"/>
     </joint>
+    <!-- joint3 elbow (Y): elbow motor + forearm -->
     <link name="${prefix}link3">
-      <visual><origin rpy="${pi2} 0 0"/>
-        <geometry><cylinder radius="0.042" length="0.095"/></geometry>
-        <material name="${color}"/></visual>
-      <visual><origin xyz="0 0 ${fore/2}"/>
-        <geometry><box size="0.045 0.045 ${fore}"/></geometry>
-        <material name="wc_link"/></visual>
-      <collision><origin xyz="0 0 ${fore/2}"/>
-        <geometry><box size="0.045 0.045 ${fore}"/></geometry></collision>
-      <xacro:ibox mass="0.6"/>
+      <xacro:wc_motor radius="0.042" ln="0.095" rpy="${pi2} 0 0" mat="${color}"/>
+      <xacro:wc_seg w="0.045" ln="${fore}"/>
+      <xacro:wc_inertia mass="0.6"/>
     </link>
     <joint name="${prefix}joint3" type="revolute">
@@ -80,13 +89,9 @@
       <limit lower="-${jl}" upper="${jl}" effort="20" velocity="2.0"/>
     </joint>
+    <!-- joint4 wrist roll (Z) -->
     <link name="${prefix}link4">
-      <visual><geometry><cylinder radius="0.036" length="0.07"/></geometry>
-        <material name="wc_joint"/></visual>
-      <visual><origin xyz="0 0 ${wrist/2}"/>
-        <geometry><box size="0.04 0.04 ${wrist}"/></geometry>
-        <material name="wc_link"/></visual>
-      <collision><origin xyz="0 0 ${wrist/2}"/>
-        <geometry><box size="0.04 0.04 ${wrist}"/></geometry></collision>
-      <xacro:ibox mass="0.3"/>
+      <xacro:wc_motor radius="0.036" ln="0.07"/>
+      <xacro:wc_seg w="0.04" ln="${wrist}"/>
+      <xacro:wc_inertia mass="0.3"/>
     </link>
     <joint name="${prefix}joint4" type="revolute">
@@ -95,9 +100,9 @@
       <limit lower="-${jl}" upper="${jl}" effort="10" velocity="2.5"/>
     </joint>
+    <!-- joint5 wrist pitch (Y) -->
     <link name="${prefix}link5">
-      <visual><origin rpy="${pi2} 0 0"/>
-        <geometry><cylinder radius="0.034" length="0.07"/></geometry>
-        <material name="${color}"/></visual>
-      <xacro:ibox mass="0.2"/>
+      <xacro:wc_motor radius="0.034" ln="0.07" rpy="${pi2} 0 0" mat="${color}"/>
+      <xacro:wc_seg w="0.035" ln="0.05"/>
+      <xacro:wc_inertia mass="0.2"/>
     </link>
     <joint name="${prefix}joint5" type="revolute">
@@ -106,17 +111,16 @@
       <limit lower="-${jl}" upper="${jl}" effort="10" velocity="2.5"/>
     </joint>
-    <!-- tool0 flange + a welding torch (neck + copper nozzle) -->
+    <!-- joint6 tool roll (Z): flange + welding torch -->
     <link name="${prefix}tool0">
-      <visual><geometry><cylinder radius="0.03" length="0.03"/></geometry>
-        <material name="wc_joint"/></visual>
-      <visual><origin xyz="0 0 0.06"/>
+      <xacro:wc_motor radius="0.03" ln="0.03"/>
+      <visual><origin xyz="0 0 0.07"/>
         <geometry><cylinder radius="0.014" length="0.10"/></geometry>
         <material name="wc_torch"/></visual>
-      <visual><origin xyz="0 0 0.13"/>
+      <visual><origin xyz="0 0 0.14"/>
         <geometry><cylinder radius="0.022" length="0.04"/></geometry>
         <material name="wc_copper"/></visual>
-      <collision><origin xyz="0 0 0.07"/>
-        <geometry><cylinder radius="0.03" length="0.16"/></geometry></collision>
-      <xacro:ibox mass="0.2"/>
+      <collision><origin xyz="0 0 0.08"/>
+        <geometry><cylinder radius="0.03" length="0.18"/></geometry></collision>
+      <xacro:wc_inertia mass="0.2"/>
     </link>
     <joint name="${prefix}joint6" type="revolute">
@@ -125,5 +129,4 @@
       <limit lower="-${jl}" upper="${jl}" effort="10" velocity="2.5"/>
     </joint>
-    <!-- ros2_control system for this arm (mock hardware) -->
     <ros2_control name="${prefix}hw" type="system">
       <hardware><plugin>mock_components/GenericSystem</plugin></hardware>
