Commit message: weld_cell: fix arm directions/positions — torches now reach the seams
- root cause: hand-tuned welding poses folded the arms BACKWARD (negative
  shoulder), torches sat next to their own bases instead of reaching in
- tools/arm_ik.py: pure-python FK + coordinate-descent IK (no ROS) — solves
  torch-down poses; found the straight-down reach is ~0.25 fwd/up (further
  is unreachable once the torch must lift vertical)
- coordinator uses the IK poses; joint1 sweeps the seam
- car part lowered (seams at z=0.25) + arms moved to 0.25 in front of each
  seam so the reach lands on the workpiece
- verified: torch tips at seam height 0.246 on the correct rails

Co-Authored-By: Claude Fable 5 <noreply@anthropic.com>

File: ros2/weld_cell/urdf/multi_weld_cell.urdf.xacro (robot description, xacro)
@@ -8,25 +8,27 @@
   <material name="fixture"><color rgba="0.25 0.26 0.28 1"/></material>
   <link name="world"/>
-  <!-- ===== the car part: an underbody floor pan on a fixture ===== -->
+  <!-- ===== the car part: an underbody floor pan on a low fixture =====
+       Seams sit at z=0.25 so the floor-mounted arms reach them torch-down.
+       Rails at y=+/-0.13, cross member at x=0.13. -->
   <link name="car_part">
-    <!-- floor pan -->
-    <visual><origin xyz="0 0 0.40"/>
-      <geometry><box size="0.55 0.40 0.02"/></geometry>
+    <!-- floor pan (top at z=0.25) -->
+    <visual><origin xyz="0 0 0.24"/>
+      <geometry><box size="0.32 0.28 0.02"/></geometry>
       <material name="car_body"/></visual>
-    <!-- left side rail (seam #1 where it meets the floor) -->
-    <visual><origin xyz="0 0.17 0.45"/>
-      <geometry><box size="0.55 0.03 0.10"/></geometry>
+    <!-- left side rail (seam #1) -->
+    <visual><origin xyz="0 0.13 0.29"/>
+      <geometry><box size="0.32 0.03 0.08"/></geometry>
       <material name="car_body"/></visual>
     <!-- right side rail (seam #2) -->
-    <visual><origin xyz="0 -0.17 0.45"/>
-      <geometry><box size="0.55 0.03 0.10"/></geometry>
+    <visual><origin xyz="0 -0.13 0.29"/>
+      <geometry><box size="0.32 0.03 0.08"/></geometry>
       <material name="car_body"/></visual>
     <!-- cross member (seam #3) -->
-    <visual><origin xyz="0.18 0 0.45"/>
-      <geometry><box size="0.03 0.40 0.10"/></geometry>
+    <visual><origin xyz="0.13 0 0.29"/>
+      <geometry><box size="0.03 0.28 0.08"/></geometry>
       <material name="car_body"/></visual>
-    <!-- fixture legs -->
-    <visual><origin xyz="0 0 0.20"/>
-      <geometry><box size="0.5 0.35 0.4"/></geometry>
+    <!-- fixture -->
+    <visual><origin xyz="0 0 0.115"/>
+      <geometry><box size="0.26 0.22 0.23"/></geometry>
       <material name="fixture"/></visual>
     <inertial><mass value="20"/>
@@ -36,13 +38,13 @@
     <parent link="world"/><child link="car_part"/>
   </joint>
-  <!-- ===== three welding robots around the part ===== -->
-  <!-- arm1: left side, welds the left rail seam -->
+  <!-- ===== three welding robots, each 0.25 in front of its seam ===== -->
+  <!-- arm1: welds the left rail (world +y) -->
   <xacro:weld_arm prefix="arm1_" parent="world"
-                  x="0.0" y="0.62" z="0.0" yaw="-1.5708" color="wc_accent"/>
-  <!-- arm2: right side, welds the right rail seam -->
+                  x="0.0" y="0.38" z="0.0" yaw="-1.5708" color="wc_accent"/>
+  <!-- arm2: welds the right rail (world -y) -->
   <xacro:weld_arm prefix="arm2_" parent="world"
-                  x="0.0" y="-0.62" z="0.0" yaw="1.5708" color="wc_accent"/>
-  <!-- arm3: front, welds the cross member -->
+                  x="0.0" y="-0.38" z="0.0" yaw="1.5708" color="wc_accent"/>
+  <!-- arm3: welds the cross member (world +x) -->
   <xacro:weld_arm prefix="arm3_" parent="world"
-                  x="0.66" y="0.0" z="0.0" yaw="3.1416" color="wc_accent"/>
+                  x="0.38" y="0.0" z="0.0" yaw="3.1416" color="wc_accent"/>
 </robot>

Commit message: weld_cell: collision-check the trajectories, fix the self-collision found
- tools/check_trajectory.py: interpolates the full 3-arm weld cycle and
  checks every state via /check_state_validity (self + inter-arm + car-part)
- it CAUGHT a real bug: the IK weld pose cranked the wrist (j5=2.44) so the
  torch (tool0) folded into the forearm (link3) — tool0<->link3 collision
- fix: arm_ik.py regularizes toward a natural posture + a down-forward reach
  (arms on 0.30m pedestals reach DOWN onto the seam); new pose uses the elbow
  (j3=1.39) with a moderate wrist (j5=0.96), torch straight down, cost 0.0
- weld_arm.xacro: optional pedestal (ped param); arms repositioned
- re-verified: all 55 trajectory states COLLISION-FREE

Co-Authored-By: Claude Fable 5 <noreply@anthropic.com>

File: ros2/weld_cell/urdf/multi_weld_cell.urdf.xacro (robot description, xacro)
@@ -38,13 +38,14 @@
     <parent link="world"/><child link="car_part"/>
   </joint>
-  <!-- ===== three welding robots, each 0.25 in front of its seam ===== -->
+  <!-- ===== three welding robots on 0.30 m pedestals, each 0.30 in front
+       of its seam, reaching DOWN-forward onto the part ===== -->
   <!-- arm1: welds the left rail (world +y) -->
   <xacro:weld_arm prefix="arm1_" parent="world"
-                  x="0.0" y="0.38" z="0.0" yaw="-1.5708" color="wc_accent"/>
+                  x="0.0" y="0.43" z="0.30" yaw="-1.5708" color="wc_accent" ped="0.30"/>
   <!-- arm2: welds the right rail (world -y) -->
   <xacro:weld_arm prefix="arm2_" parent="world"
-                  x="0.0" y="-0.38" z="0.0" yaw="1.5708" color="wc_accent"/>
+                  x="0.0" y="-0.43" z="0.30" yaw="1.5708" color="wc_accent" ped="0.30"/>
   <!-- arm3: welds the cross member (world +x) -->
   <xacro:weld_arm prefix="arm3_" parent="world"
-                  x="0.38" y="0.0" z="0.0" yaw="3.1416" color="wc_accent"/>
+                  x="0.43" y="0.0" z="0.30" yaw="3.1416" color="wc_accent" ped="0.30"/>
 </robot>

File: ros2/weld_cell/urdf/weld_arm.xacro (robot description, xacro)
@@ -31,5 +31,5 @@
     </inertial>
   </xacro:macro>
-  <xacro:macro name="weld_arm" params="prefix parent x y z yaw color:=wc_accent">
+  <xacro:macro name="weld_arm" params="prefix parent x y z yaw color:=wc_accent ped:=0.0">
     <xacro:property name="pi2" value="1.5708"/>
     <xacro:property name="waist_h" value="0.08"/>
@@ -42,6 +42,13 @@
       <origin xyz="${x} ${y} ${z}" rpy="0 0 ${yaw}"/>
     </joint>
-    <!-- ribbed base + riser -->
+    <!-- ribbed base + riser (+ pedestal down to the floor if ped>0) -->
     <link name="${prefix}base_link">
+      <xacro:if value="${ped > 0}">
+        <visual><origin xyz="0 0 ${-ped/2}"/>
+          <geometry><cylinder radius="0.07" length="${ped}"/></geometry>
+          <material name="wc_joint"/></visual>
+        <collision><origin xyz="0 0 ${-ped/2}"/>
+          <geometry><cylinder radius="0.07" length="${ped}"/></geometry></collision>
+      </xacro:if>
       <visual><origin xyz="0 0 0.015"/>
         <geometry><cylinder radius="0.08" length="0.03"/></geometry>
